Commit message: realsense

File: ibrain/urdf/ibrain.xacro (robot description, xacro)
@@ -1,6 +1,5 @@
 <?xml version="1.0" ?>
 <robot name="ibrain" xmlns:xacro="https://www.ros.org/wiki/xacro" >
-  <xacro:include filename="$(find warehouse_bot)/gazebo/whbot_physics.gazebo"/>
-  <xacro:include filename="$(find warehouse_bot)/urdf/_d435.urdf.xacro" />
+  <xacro:include filename="$(find ibrain)/urdf/_d435.urdf.xacro" />
   <gazebo reference="link_chassis">
     <material>Gazebo/Orange</material>
@@ -217,4 +216,7 @@
     <joint_properties damping="1.0" friction="1.0" />
   </joint>
+  <sensor_d435 parent="upper_body">
+    <origin xyz="0.02 1.1e-05 0.08" rpy="0 0 0"/>
+  </sensor_d435>
 <!-- inner_body -->
     <link name="inner_body">

Commit message: models

File: ibrain/urdf/ibrain.xacro (robot description, xacro)
@@ -217,5 +217,5 @@
   </joint>
   <sensor_d435 parent="upper_body">
-    <origin xyz="0.02 1.1e-05 0.08" rpy="0 0 0"/>
+    <origin xyz="0.0 0.0 0.35" rpy="0 0 0"/>
   </sensor_d435>
 <!-- inner_body -->
@@ -324,7 +324,7 @@
 		</plugin>
 	</gazebo>
-  	<!--Lidar2-->
+  	<!--Lidar1-->
 	<gazebo reference="sensor_laser1">
-		<sensor type="ray" name="head_hokuyo_sensor">
+		<sensor type="ray" name="head_hokuyo_sensor1">
 			<pose>0 0 0 0 0 0</pose>
 			<visualize>false</visualize>
@@ -356,7 +356,7 @@
 		</sensor>
 	</gazebo>
-  	<!--Lidar2
+  	<!--Lidar2 -->
 	<gazebo reference="sensor_laser2">
-		<sensor type="ray" name="head_hokuyo_sensor">
+		<sensor type="ray" name="head_hokuyo_sensor2">
 			<pose>0 0 0 0 0 0</pose>
 			<visualize>false</visualize>
@@ -367,6 +367,6 @@
 						<samples>720</samples>
 						<resolution>1</resolution>
-						<min_angle>-1.5</min_angle>
-						<max_angle>1.5</max_angle>
+						<min_angle>1.5</min_angle>
+						<max_angle>-1.5</max_angle>
 					</horizontal>
 				</scan>
@@ -387,4 +387,4 @@
 			</plugin>
 		</sensor>
-	</gazebo>  -->
+	</gazebo>
 </robot>

Commit message: alignment changes

File: ibrain/urdf/ibrain.xacro (robot description, xacro)
@@ -217,5 +217,5 @@
   </joint>
   <sensor_d435 parent="upper_body">
-    <origin xyz="0.0 0.0 0.35" rpy="0 0 0"/>
+    <origin xyz="0.05 0.0 -0.36" rpy="0 0 0"/>
   </sensor_d435>
 <!-- inner_body -->
@@ -272,30 +272,4 @@
     <parent link="link_chassis"/>
     <child link="sensor_laser1"/>
-  </joint>
- <!-- Lidar2 -->
-   <link name="sensor_laser2">
-    <inertial>
-      <origin xyz="0 0 0" rpy="0 0 0" />
-      <mass value="1" />
-      <!-- RANDOM INERTIA BELOW -->
-      <inertia ixx="0.02" ixy="0" ixz="0" iyy="0.02" iyz="0" izz="0.02"/>
-    </inertial>
-    <visual>
-      <origin xyz="0 0 0" rpy="0 0 0" />
-      <geometry>
-        <cylinder radius="0.05" length="0.1"/>
-      </geometry>
-    </visual>
-    <collision>
-      <origin xyz="0 0 0" rpy="0 0 0"/>
-      <geometry>
-        <cylinder radius="0.05" length="0.1"/>
-      </geometry>
-    </collision>
-  </link>
-  <joint name="joint_sensor_laser2" type="fixed">
-    <origin xyz="-0.15 0 0.1" rpy="0 0 0"/>
-    <parent link="link_chassis"/>
-    <child link="sensor_laser2"/>
   </joint>
 	<gazebo>
@@ -341,5 +315,5 @@
 				<range>
 					<min>0.15</min>
-					<max>12.0</max>
+					<max>8.0</max>
 					<resolution>0.01</resolution>
 				</range>
@@ -356,35 +330,3 @@
 		</sensor>
 	</gazebo>
-  	<!--Lidar2 -->
-	<gazebo reference="sensor_laser2">
-		<sensor type="ray" name="head_hokuyo_sensor2">
-			<pose>0 0 0 0 0 0</pose>
-			<visualize>false</visualize>
-			<update_rate>10</update_rate>
-			<ray>
-				<scan>
-					<horizontal>
-						<samples>720</samples>
-						<resolution>1</resolution>
-						<min_angle>1.5</min_angle>
-						<max_angle>-1.5</max_angle>
-					</horizontal>
-				</scan>
-				<range>
-					<min>0.15</min>
-					<max>12.0</max>
-					<resolution>0.01</resolution>
-				</range>
-				<noise>
-					<type>gaussian</type>
-					<mean>0.0</mean>
-					<stddev>0.01</stddev>
-				</noise>
-			</ray>
-			<plugin name="gazebo_ros_head_hokuyo_controller" filename="libgazebo_ros_laser.so">
-				<topicName>/wh_base/laser/scan2</topicName>
-				<frameName>sensor_laser2</frameName>
-			</plugin>
-		</sensor>
-	</gazebo>
 </robot>

Commit message: slam

File: ibrain/urdf/ibrain.xacro (robot description, xacro)
@@ -27,5 +27,5 @@
     <pose>0 0 0.1 0 0 0</pose>
     <inertial>
-      <mass value="5"/>
+      <mass value="50"/>
       <origin rpy="0 0 0" xyz="0 0 0.1"/>
       <inertia ixx="0.0395416666667" ixy="0" ixz="0" iyy="0.106208333333" iyz="0" izz="0.106208333333"/>
@@ -33,11 +33,11 @@
     <collision name="collision_chassis">
       <geometry>
-        <box size="0.4 0.4 0.1"/>
-      </geometry>
-    </collision>
-    <visual>
-      <origin rpy="0 0 0" xyz="0 0 0"/>
-      <geometry>
-        <box size="0.4 0.4 0.1"/>
+        <box size="0.4 0.4 0.05"/>
+      </geometry>
+    </collision>
+    <visual>
+      <origin rpy="0 0 0" xyz="0 0 0"/>
+      <geometry>
+        <box size="0.4 0.4 0.05"/>
       </geometry>
       <material name="blue"/>
@@ -54,5 +54,5 @@
       <origin rpy="0 1.5707 1.5707" xyz="0 0 0" />
       <geometry>
-        <cylinder length="0.04" radius="0.08"/>
+        <cylinder length="0.04" radius="0.05"/>
       </geometry>
     </collision>
@@ -60,5 +60,5 @@
       <origin rpy="0 1.5707 1.5707" xyz="0 0 0"/>
       <geometry>
-        <cylinder length="0.04" radius="0.08"/>
+        <cylinder length="0.04" radius="0.05"/>
       </geometry>
     </visual>
@@ -82,5 +82,5 @@
       <origin rpy="0 1.5707 1.5707" xyz="0 0 0" />
       <geometry>
-        <cylinder length="0.04" radius="0.08"/>
+        <cylinder length="0.04" radius="0.05"/>
       </geometry>
     </collision>
@@ -88,5 +88,5 @@
       <origin rpy="0 1.5707 1.5707" xyz="0 0 0"/>
       <geometry>
-        <cylinder length="0.04" radius="0.08"/>
+        <cylinder length="0.04" radius="0.05"/>
       </geometry>
     </visual>
@@ -111,5 +111,5 @@
       <origin rpy="0 1.5707 1.5707" xyz="0 0 0" />
       <geometry>
-        <cylinder length="0.04" radius="0.08"/>
+        <cylinder length="0.04" radius="0.05"/>
       </geometry>
     </collision>
@@ -117,5 +117,5 @@
       <origin rpy="0 1.5707 1.5707" xyz="0 0 0"/>
       <geometry>
-        <cylinder length="0.04" radius="0.08"/>
+        <cylinder length="0.04" radius="0.05"/>
       </geometry>
     </visual>
@@ -140,5 +140,5 @@
       <origin rpy="0 1.5707 1.5707" xyz="0 0 0" />
       <geometry>
-        <cylinder length="0.04" radius="0.08"/>
+        <cylinder length="0.04" radius="0.05"/>
       </geometry>
     </collision>
@@ -146,5 +146,5 @@
       <origin rpy="0 1.5707 1.5707" xyz="0 0 0"/>
       <geometry>
-        <cylinder length="0.04" radius="0.08"/>
+        <cylinder length="0.04" radius="0.05"/>
       </geometry>
     </visual>
@@ -163,5 +163,5 @@
     <pose>0 0 0.1 0 0 0</pose>
     <inertial>
-      <mass value="5"/>
+      <mass value="20"/>
       <origin rpy="0 0 0" xyz="0 0 0"/>
       <inertia ixx="0.0395416666667" ixy="0" ixz="0" iyy="0.106208333333" iyz="0" izz="0.106208333333"/>
@@ -273,7 +273,7 @@
     <child link="sensor_laser1"/>
   </joint>
-	<gazebo>
+ <gazebo>
 		<plugin filename="libgazebo_ros_control.so" name="gazebo_ros_control">
-			<robotNamespace>/ibrain</robotNamespace>
+			<robotNamespace>/</robotNamespace>
 			<robotSimType>gazebo_ros_control/DefaultRobotHWSim</robotSimType>
 			<legacyModeNS>true</legacyModeNS>
@@ -285,8 +285,8 @@
 			<alwaysOn>true</alwaysOn>
 			<updateRate>20</updateRate>
-			<leftJoint>joint_left_wheel</leftJoint>
-      <leftJoint>joint_left_wheel2</leftJoint>
-			<rightJoint>joint_right_wheel</rightJoint>
-    	<rightJoint>joint_right_wheel2</rightJoint>
+			<leftJoint>joint_right_wheel</leftJoint>
+      <leftJoint>joint_right_wheel2</leftJoint>
+			<rightJoint>joint_left_wheel</rightJoint>
+    	<rightJoint>joint_left_wheel2</rightJoint>
 			<wheelSeparation>0.53</wheelSeparation>
 			<wheelDiameter>0.1524</wheelDiameter>
@@ -295,5 +295,5 @@
 			<odometryFrame>odom</odometryFrame>
 			<robotBaseFrame>link_chassis</robotBaseFrame>
-      <robotNamespace>/ibrain</robotNamespace>
+      <robotNamespace>/</robotNamespace>
 		</plugin>
 	</gazebo>
@@ -325,5 +325,5 @@
 			</ray>
 			<plugin name="gazebo_ros_head_hokuyo_controller" filename="libgazebo_ros_laser.so">
-				<topicName>/wh_base/laser/scan1</topicName>
+				<topicName>/scan1</topicName>
 				<frameName>sensor_laser1</frameName>
 			</plugin>

Commit message: rtab

File: ibrain/urdf/ibrain.xacro (robot description, xacro)
@@ -1,5 +1,5 @@
 <?xml version="1.0" ?>
 <robot name="ibrain" xmlns:xacro="https://www.ros.org/wiki/xacro" >
-  <xacro:include filename="$(find ibrain)/urdf/_d435.urdf.xacro" />
+  <!-- <xacro:include filename="$(find ibrain)/urdf/kinect_camera.urdf.xacro" /> -->
   <gazebo reference="link_chassis">
     <material>Gazebo/Orange</material>
@@ -216,7 +216,7 @@
     <joint_properties damping="1.0" friction="1.0" />
   </joint>
-  <sensor_d435 parent="upper_body">
+  <!-- <kinect_camera parent="upper_body" name="camera">
     <origin xyz="0.05 0.0 -0.36" rpy="0 0 0"/>
-  </sensor_d435>
+  </kinect_camera> -->
 <!-- inner_body -->
     <link name="inner_body">
@@ -331,5 +331,5 @@
 	</gazebo>
   <!-- imu -->
-    <gazebo>
+    <!-- <gazebo>
     <plugin name="imu_plugin" filename="libgazebo_ros_imu.so">
       <alwaysOn>true</alwaysOn>
@@ -340,4 +340,79 @@
       <updateRate>20.0</updateRate>
     </plugin>
-  </gazebo>
+  </gazebo> -->
+<joint name="camera_joint" type="fixed">
+        <parent link="upper_body"/>
+        <child link="camera_link"/>
+      </joint>
+      <link name="camera_link">
+        <inertial_sphere mass="0.01" diameter="0.07" />
+        <visual>
+          <origin xyz="0 0 0" rpy="0 0 0" />
+          <geometry>
+            <mesh filename="package://ibrain/meshes/kinect.dae"/>
+          </geometry>
+        </visual>
+        <collision>
+          <origin xyz="0 0 0" rpy="0 0 0" />
+          <geometry>
+            <mesh filename="package://ibrain/meshes/kinect.dae"/>
+          </geometry>
+        </collision>
+      </link>
+      <joint name="camera_depth_joint" type="fixed">
+        <origin xyz="0.0 -0.02 0.0" rpy="0 0 0" />
+        <parent link="camera_link" />
+        <child link="camera_depth_frame"/>
+      </joint>
+      <link name="camera_depth_frame"/>
+      <joint name="camera_depth_optical_joint" type="fixed">
+        <origin xyz="0 0 0" rpy="${-3.14/2} 0.0 ${-3.14/2}" />
+        <parent link="camera_depth_frame" />
+        <child link="camera_depth_optical_frame"/>
+      </joint>
+      <link name="camera_depth_optical_frame"/>
+      <joint name="camera_rgb_joint" type="fixed">
+        <origin xyz="0.0 -0.0125 0.0" rpy="0 0 0" />
+        <parent link="camera_link" />
+        <child link="camera_rgb_frame"/>
+      </joint>
+      <link name="camera_rgb_frame"/>
+      <joint name="camera_rgb_optical_joint" type="fixed">
+        <origin xyz="0 0 0" rpy="${-3.14/2} 0.0 ${-3.14/2}" />
+        <parent link="camera_rgb_frame" />
+        <child link="camera_rgb_optical_frame"/>
+      </joint>
+      <link name="camera_rgb_optical_frame"/>
+      <gazebo reference="camera_depth_frame">
+        <sensor type="depth" name="camera">
+          <update_rate>20</update_rate>
+          <camera>
+            <horizontal_fov>${60 * 3.14/180.0}</horizontal_fov>
+            <image>
+              <format>R8G8B8</format>
+              <width>640</width>
+              <height>480</height>
+            </image>
+            <clip>
+              <near>0.05</near>
+              <far>3</far>
+            </clip>
+          </camera>
+          <plugin name="camera_camera_controller" filename="libgazebo_ros_openni_kinect.so">
+            <alwaysOn>true</alwaysOn>
+            <updateRate>20</updateRate>
+            <imageTopicName>camera/rgb/image_raw</imageTopicName>
+            <cameraInfoTopicName>camera/rgb/camera_info</cameraInfoTopicName>
+            <depthImageTopicName>camera/depth/image_raw</depthImageTopicName>
+            <depthImageCameraInfoTopicName>camera/depth/camera_info</depthImageCameraInfoTopicName>
+            <pointCloudTopicName>camera/depth/points</pointCloudTopicName>
+            <frameName>camera_depth_optical_frame</frameName>
+            <distortion_k1>0.0</distortion_k1>
+            <distortion_k2>0.0</distortion_k2>
+            <distortion_k3>0.0</distortion_k3>
+            <distortion_t1>0.0</distortion_t1>
+            <distortion_t2>0.0</distortion_t2>
+          </plugin>
+        </sensor>
+      </gazebo>
 </robot>
